File: MP1Flight.sch (KiCad schematic (older format))
At the start: 46 parts, among them J1 Conn_ARM_JTAG_SWD_10, J3 Conn_01x06_Female, J4 Conn_01x06_Female, J5 Conn_01x04_Female, J6 Conn_01x04_Male, J6 Conn_01x06_Female, J7 Screw_Terminal_01x02, SW1 SW_Push, U2 VisionSOM-STM32MP1, U3 74LVC2G86

Commit message: adding in SD card with power switch
Parts:
- added C19, C22, C24: 10uF, symbol Device:C
- added C20: 1uF, symbol Device:C
- added C21: 100nF, Capacitor_SMD:C_0603_1608Metric_Pad1.05x0.95mm_HandSolder, symbol Device:C
- added C23, C25: 100nF, symbol Device:C
- added J?: Micro_SD_Card_Det, symbol Connector:Micro_SD_Card_Det
- added R8: 12k, Resistor_SMD:R_0603_1608Metric_Pad1.05x0.95mm_HandSolder, symbol Device:R
- added R9: 10k, symbol Device:R
- added SS1: BD2242G-GTR, SOT95P280X125-6N, symbol BD2242G-GTR:BD2242G-GTR
- added Z1: 1SMA5919BT3G, DIOM5226X220N, symbol 1SMA5919BT3G:1SMA5919BT3G
- C6: value 0.1uF -> 100uF
- gave numbers to parts that had none: 3
Connections:
- net +3V3: now also C19.1, C20.1, SS1.1 (IN)
- net +5V: now also D2.4, Z1.1
- net ABAT: now also U2.157 (GPIO-PA1)
- net GND: now also C19.2, C20.2, C21.2, C22.2, C23.2, C24.2, C25.2, J?.11 (SHIELD), J?.6 (VSS), R8.2, R9.2, SS1.2 (GND), Z1.2
- net MPU9250_CS: now also U2.55 (GPIO-PC0)
- net MPU9250_DRDY: now also U2.58 (GPIO-PB1)
- net MPU9250_MISO: now also U2.119 (GPIO-PC2)
- net MPU9250_MOSI: now also U2.47 (GPIO-PC3)
- net MPU9250_SCLK: now also U2.129 (LCD-R5)
- net STM32-NRST: now also SS1.3 (EN)
- new net: R9.1, SS1.4 (/OC)
- new net: R8.1, SS1.5 (ILIM)
- new net VDD_SDCARD: C21.1, C22.1, C23.1, C24.1, C25.1, J?.4 (VDD), SS1.6 (OUT)
Other:
- moved on the sheet: C6, D2, F1, F2, J7, TP1

Commit message: Moved connectors to child sheet
Parts:
- removed C10, C17: 2u2, symbol Device:C
- removed C15, C16, C4: 100nF, Capacitor_SMD:C_0603_1608Metric_Pad1.05x0.95mm_HandSolder, symbol Device:C
- removed C18: 100uF, symbol Device:C
- removed J1: Conn_ARM_JTAG_SWD_10, FTSH-105-01-L-DV-K-P-TR:FTSH10501LDVKPTR, symbol Connector:Conn_ARM_JTAG_SWD_10
- removed J3, J4, J6: Conn_01x06_Female, symbol Connector:Conn_01x06_Female
- removed J5: Conn_01x04_Female, symbol Connector:Conn_01x04_Female
- removed JP1: SolderJumper_3_Bridged12, Jumper:SolderJumper-3_P1.3mm_Bridged12_RoundedPad1.0x1.5mm_NumberLabels, symbol Jumper:SolderJumper_3_Bridged12
- removed R11: 2k2, Resistor_SMD:R_0603_1608Metric_Pad1.05x0.95mm_HandSolder, symbol Device:R
- removed R12: 2K2, Resistor_SMD:R_0603_1608Metric_Pad1.05x0.95mm_HandSolder, symbol Device:R
- removed U3: 74LVC2G86, SN74LVC2G86DCTR:SOP65P400X130-8N, symbol 74xGxx:74LVC2G86
- gave numbers to parts that had none: 1
- renumbered C19 to C14, C20 to C15, R7 to R4
Connections:
- net labels removed: FRSKY_IN, FRSKY_INV, FRSKY_OUT
- wire segments 201 -> 152
Other:
- note added: "LCD NOT BEING USED"
- note removed: "Basic GPS Port\n\n"
- note removed: "DEBUG Connector\n"
- note removed: "Telemetry 1\n"
- note removed: "USART1\n"
- note removed: "USART3\n\n"
- note removed: "Unsure about which net to use\n"
