File: ServoConnectors.sch (KiCad schematic (older format))
At the start: 6 parts, among them M1 Motor_Servo, M2 Motor_Servo, M3 Motor_Servo, M4 Motor_Servo, M5 Motor_Servo, M6 Motor_Servo

Commit message: Added in Buzzer and N channel mosfet
Parts:
- removed M1, M2, M3, M4, M5, M6: Motor_Servo, Connector_PinHeader_2.54mm:PinHeader_1x03_P2.54mm_Vertical, symbol Motor:Motor_Servo
- added M1: Servo_Connector, symbol ServoConnector3_6:Servo_Connector
Changed lines of the file:
@@
 $Descr A4 11693 8268
 encoding utf-8
-Sheet 7 7
+Sheet 6 7
 Title "Servo Connectors"
 Date ""
@@
 $EndDescr
 $Comp
-L Motor:Motor_Servo M1
-U 1 1 5F0832E9
-P 5250 2350
-F 0 "M1" H 5582 2415 50  0000 L CNN
-F 1 "Motor_Servo" H 5582 2324 50  0000 L CNN
-F 2 "Connector_PinHeader_2.54mm:PinHeader_1x03_P2.54mm_Vertical" H 5250 2160 50  0001 C CNN
-F 3 "http://forums.parallax.com/uploads/attachments/46831/74481.png" H 5250 2160 50  0001 C CNN
-	1    5250 2350
-	1    0    0    -1
-$EndComp
-$Comp
-L Motor:Motor_Servo M2
-U 1 1 5F084478
-P 5250 2750
-F 0 "M2" H 5582 2815 50  0000 L CNN
-F 1 "Motor_Servo" H 5582 2724 50  0000 L CNN
-F 2 "Connector_PinHeader_2.54mm:PinHeader_1x03_P2.54mm_Vertical" H 5250 2560 50  0001 C CNN
-F 3 "http://forums.parallax.com/uploads/attachments/46831/74481.png" H 5250 2560 50  0001 C CNN
-	1    5250 2750
-	1    0    0    -1
-$EndComp
-$Comp
-L Motor:Motor_Servo M3
-U 1 1 5F084FE9
-P 5250 3150
-F 0 "M3" H 5582 3215 50  0000 L CNN
-F 1 "Motor_Servo" H 5582 3124 50  0000 L CNN
-F 2 "Connector_PinHeader_2.54mm:PinHeader_1x03_P2.54mm_Vertical" H 5250 2960 50  0001 C CNN
-F 3 "http://forums.parallax.com/uploads/attachments/46831/74481.png" H 5250 2960 50  0001 C CNN
-	1    5250 3150
-	1    0    0    -1
-$EndComp
-$Comp
-L Motor:Motor_Servo M5
-U 1 1 5F086780
-P 5250 3950
-F 0 "M5" H 5582 4015 50  0000 L CNN
-F 1 "Motor_Servo" H 5582 3924 50  0000 L CNN
-F 2 "Connector_PinHeader_2.54mm:PinHeader_1x03_P2.54mm_Vertical" H 5250 3760 50  0001 C CNN
-F 3 "http://forums.parallax.com/uploads/attachments/46831/74481.png" H 5250 3760 50  0001 C CNN
-	1    5250 3950
-	1    0    0    -1
-$EndComp
-$Comp
-L Motor:Motor_Servo M6
-U 1 1 5F0876B5
-P 5250 4350
-F 0 "M6" H 5582 4415 50  0000 L CNN
-F 1 "Motor_Servo" H 5582 4324 50  0000 L CNN
-F 2 "Connector_PinHeader_2.54mm:PinHeader_1x03_P2.54mm_Vertical" H 5250 4160 50  0001 C CNN
-F 3 "http://forums.parallax.com/uploads/attachments/46831/74481.png" H 5250 4160 50  0001 C CNN
-	1    5250 4350
-	1    0    0    -1
-$EndComp
-$Comp
 L power:GND #PWR022
 U 1 1 5F08D973
-P 4950 2850
-F 0 "#PWR022" H 4950 2600 50  0001 C CNN
-F 1 "GND" V 4955 2722 50  0000 R CNN
-F 2 "" H 4950 2850 50  0001 C CNN
-F 3 "" H 4950 2850 50  0001 C CNN
-	1    4950 2850
+P 5100 2950
+F 0 "#PWR022" H 5100 2700 50  0001 C CNN
+F 1 "GND" V 5105 2822 50  0000 R CNN
+F 2 "" H 5100 2950 50  0001 C CNN
+F 3 "" H 5100 2950 50  0001 C CNN
+	1    5100 2950
 	0    1    1    0
 $EndComp
@@
 L power:GND #PWR021
 U 1 1 5F08E6E0
-P 4950 2450
-F 0 "#PWR021" H 4950 2200 50  0001 C CNN
-F 1 "GND" V 4955 2322 50  0000 R CNN
-F 2 "" H 4950 2450 50  0001 C CNN
-F 3 "" H 4950 2450 50  0001 C CNN
-	1    4950 2450
+P 5100 2650
+F 0 "#PWR021" H 5100 2400 50  0001 C CNN
+F 1 "GND" V 5100 2550 50  0000 R CNN
+F 2 "" H 5100 2650 50  0001 C CNN
+F 3 "" H 5100 2650 50  0001 C CNN
+	1    5100 2650
 	0    1    1    0
 $EndComp
@@
 L power:GND #PWR023
 U 1 1 5F08EDEA
-P 4950 3250
-F 0 "#PWR023" H 4950 3000 50  0001 C CNN
-F 1 "GND" V 4955 3122 50  0000 R CNN
-F 2 "" H 4950 3250 50  0001 C CNN
-F 3 "" H 4950 3250 50  0001 C CNN
-	1    4950 3250
+P 5100 3250
+F 0 "#PWR023" H 5100 3000 50  0001 C CNN
+F 1 "GND" V 5105 3122 50  0000 R CNN
+F 2 "" H 5100 3250 50  0001 C CNN
+F 3 "" H 5100 3250 50  0001 C CNN
+	1    5100 3250
 	0    1    1    0
-$EndComp
-$Comp
-L Motor:Motor_Servo M4
-U 1 1 5F0858B9
-P 5250 3550
-F 0 "M4" H 5582 3615 50  0000 L CNN
-F 1 "Motor_Servo" H 5582 3524 50  0000 L CNN
-F 2 "Connector_PinHeader_2.54mm:PinHeader_1x03_P2.54mm_Vertical" H 5250 3360 50  0001 C CNN
-F 3 "http://forums.parallax.com/uploads/attachments/46831/74481.png" H 5250 3360 50  0001 C CNN
-	1    5250 3550
-	1    0    0    -1
 $EndComp
 $Comp
 L power:GND #PWR024
 U 1 1 5F08F8C2
-P 4950 3650
-F 0 "#PWR024" H 4950 3400 50  0001 C CNN
-F 1 "GND" V 4955 3522 50  0000 R CNN
-F 2 "" H 4950 3650 50  0001 C CNN
-F 3 "" H 4950 3650 50  0001 C CNN
-	1    4950 3650
+P 5100 3550
+F 0 "#PWR024" H 5100 3300 50  0001 C CNN
+F 1 "GND" V 5105 3422 50  0000 R CNN
+F 2 "" H 5100 3550 50  0001 C CNN
+F 3 "" H 5100 3550 50  0001 C CNN
+	1    5100 3550
 	0    1    1    0
 $EndComp
@@
 L power:GND #PWR025
 U 1 1 5F090137
-P 4950 4050
-F 0 "#PWR025" H 4950 3800 50  0001 C CNN
-F 1 "GND" V 4955 3922 50  0000 R CNN
-F 2 "" H 4950 4050 50  0001 C CNN
-F 3 "" H 4950 4050 50  0001 C CNN
-	1    4950 4050
+P 5100 3850
+F 0 "#PWR025" H 5100 3600 50  0001 C CNN
+F 1 "GND" V 5105 3722 50  0000 R CNN
+F 2 "" H 5100 3850 50  0001 C CNN
+F 3 "" H 5100 3850 50  0001 C CNN
+	1    5100 3850
 	0    1    1    0
 $EndComp
@@
 L power:GND #PWR026
 U 1 1 5F0908A2
-P 4950 4450
-F 0 "#PWR026" H 4950 4200 50  0001 C CNN
-F 1 "GND" V 4955 4322 50  0000 R CNN
-F 2 "" H 4950 4450 50  0001 C CNN
-F 3 "" H 4950 4450 50  0001 C CNN
-	1    4950 4450
+P 5100 4150
+F 0 "#PWR026" H 5100 3900 50  0001 C CNN
+F 1 "GND" V 5105 4022 50  0000 R CNN
+F 2 "" H 5100 4150 50  0001 C CNN
+F 3 "" H 5100 4150 50  0001 C CNN
+	1    5100 4150
 	0    1    1    0
 $EndComp
+Text HLabel 5100 2450 0    50   Input ~ 0
+PWM1
+Text HLabel 5100 2750 0    50   Input ~ 0
+PWM2
+Text HLabel 5100 3050 0    50   Input ~ 0
+PWM3
+Text HLabel 5100 3350 0    50   Input ~ 0
+PWM4
+Text HLabel 5100 3650 0    50   Input ~ 0
+PWM5
+Text HLabel 5100 3950 0    50   Input ~ 0
+PWM6
+$Comp
+L ServoConnector3_6:Servo_Connector M1
+U 1 1 5F0F06B9
+P 5400 2550
+F 0 "M1" H 5778 1871 50  0000 L CNN
+F 1 "Servo_Connector" H 5778 1780 50  0000 L CNN
+F 2 "" H 5400 2360 50  0001 C CNN
+F 3 "http://forums.parallax.com/uploads/attachments/46831/74481.png" H 5400 2360 50  0001 C CNN
+	1    5400 2550
+	1    0    0    -1
+$EndComp
 Wire Wire Line
-	4550 4350 4950 4350
+	5100 2550 4700 2550
 Wire Wire Line
-	4550 4350 4550 3950
+	4700 2550 4700 2850
 Wire Wire Line
-	4550 3950 4950 3950
+	4700 2850 5100 2850
 Wire Wire Line
-	4550 3950 4550 3550
+	4700 2850 4700 3150
 Wire Wire Line
-	4550 3550 4950 3550
-Connection ~ 4550 3950
+	4700 3150 5100 3150
+Connection ~ 4700 2850
 Wire Wire Line
-	4550 3550 4550 3150
+	4700 3150 4700 3450
 Wire Wire Line
-	4550 3150 4950 3150
-Connection ~ 4550 3550
+	4700 3450 5100 3450
+Connection ~ 4700 3150
 Wire Wire Line
-	4550 3150 4550 2750
+	4700 3450 4700 3750
 Wire Wire Line
-	4550 2750 4950 2750
-Connection ~ 4550 3150
+	4700 3750 5100 3750
+Connection ~ 4700 3450
 Wire Wire Line
-	4550 2750 4550 2350
+	4700 3750 4700 4050
 Wire Wire Line
-	4550 2350 4950 2350
-Connection ~ 4550 2750
-Text HLabel 4950 2250 0    50   Input ~ 0
-PWM1
-Text HLabel 4950 2650 0    50   Input ~ 0
-PWM2
-Text HLabel 4950 3050 0    50   Input ~ 0
-PWM3
-Text HLabel 4950 3450 0    50   Input ~ 0
-PWM4
-Text HLabel 4950 3850 0    50   Input ~ 0
-PWM5
-Text HLabel 4950 4250 0    50   Input ~ 0
-PWM6
+	4700 4050 5100 4050
+Connection ~ 4700 3750
 $EndSCHEMATC

Commit message: Wired up IMUs signals
Parts:
- M1: footprint (none) -> Servo3Way:3_6_2_54mm
Changed lines of the file:
@@
 F 0 "M1" H 5778 1871 50  0000 L CNN
 F 1 "Servo_Connector" H 5778 1780 50  0000 L CNN
-F 2 "" H 5400 2360 50  0001 C CNN
+F 2 "Servo3Way:3_6_2_54mm" H 5400 2360 50  0001 C CNN
 F 3 "http://forums.parallax.com/uploads/attachments/46831/74481.png" H 5400 2360 50  0001 C CNN
 	1    5400 2550
